File: Hardware/PicoPlacaClock/PicoPlacaClock.kicad_sch (KiCad schematic)
At the start: 0 parts

Commit message: arduino nano y quite backups
Parts:
- added A?: Arduino_Nano_v3.x, Module:Arduino_Nano, symbol MCU_Module:Arduino_Nano_v3.x
